File: DOMAIN-1.sch (KiCad schematic (older format))
At the start: 19 parts

Commit message: Finished matrix
Parts:
- added D? (x104): D_Small, symbol Device:D_Small
- added K_0, K_1, K_2, K_3, K_4, K_5, K_6, K_7, K_8, K_9, K_A, K_B, K_C, K_D, K_E, K_ESC, K_F, K_F1, K_F10, K_F11, K_F12, K_F2, K_F3, K_F4, K_F5, K_F6, K_F7, K_F8, K_F9, K_G, K_H, K_I, K_J, K_K, K_L, K_M, K_N, K_O, K_P, K_Q, K_R, K_S, K_T, K_U, K_V, K_W, K_X, K_Y, K_Z, K_backSlash, K_backspace, K_capsLock, K_closeBracket, K_colon, K_comma, K_decimal, K_delete, K_divide, K_down, K_eight, K_end, K_enter, K_equals, K_five, K_fn, K_four, K_home, K_insert, K_left, K_leftAlt, K_leftControl, K_leftShift, K_menu, K_multiply, K_negative, K_nine, K_numLock, K_one, K_openBracket, K_pageDown, K_pageUp, K_pause, K_period, K_printScreen, K_questionMark, K_quote, K_right, K_rightAlt, K_rightControl, K_rightShift, K_scrollLock, K_seven, K_six, K_space, K_tab, K_tallEnter, K_three, K_tilde, K_two, K_up, K_windows, K_zero, k_minus, k_plus: MX-NoLED, symbol MX_Alps_Hybrid:MX-NoLED
- added LED? (x8): WS2812B, symbol ws2812b:WS2812B
Connections:
- net +5V: now also LED?.1 (VCC), LED?.1 (VCC), LED?.1 (VCC), LED?.1 (VCC), LED?.1 (VCC), LED?.1 (VCC), LED?.1 (VCC), LED?.1 (VCC)
- net GND: now also LED?.3 (GND), LED?.3 (GND), LED?.3 (GND), LED?.3 (GND), LED?.3 (GND), LED?.3 (GND), LED?.3 (GND), LED?.3 (GND)
- new net: D?.2 (A), K_ESC.2 (ROW)
- new net: D?.2 (A), K_tilde.2 (ROW)
- new net: D?.2 (A), K_tab.2 (ROW)
- new net: D?.2 (A), K_capsLock.2 (ROW)
- new net: D?.2 (A), K_leftShift.2 (ROW)
- new net: D?.2 (A), K_leftControl.2 (ROW)
- new net: D?.2 (A), K_one.2 (ROW)
- new net: D?.2 (A), K_Q.2 (ROW)
- new net: D?.2 (A), K_A.2 (ROW)
- new net: D?.2 (A), K_Z.2 (ROW)
- new net: D?.2 (A), K_windows.2 (ROW)
- new net: D?.2 (A), K_F1.2 (ROW)
- new net: D?.2 (A), K_two.2 (ROW)
- new net: D?.2 (A), K_W.2 (ROW)
- new net: D?.2 (A), K_S.2 (ROW)
- new net: D?.2 (A), K_X.2 (ROW)
- new net: D?.2 (A), K_leftAlt.2 (ROW)
- new net: D?.2 (A), K_F2.2 (ROW)
- new net: D?.2 (A), K_three.2 (ROW)
- new net: D?.2 (A), K_E.2 (ROW)
- new net: D?.2 (A), K_D.2 (ROW)
- new net: D?.2 (A), K_C.2 (ROW)
- new net: D?.2 (A), K_F3.2 (ROW)
- new net: D?.2 (A), K_four.2 (ROW)
- new net: D?.2 (A), K_R.2 (ROW)
- new net: D?.2 (A), K_F.2 (ROW)
- new net: D?.2 (A), K_V.2 (ROW)
- new net: D?.2 (A), K_F4.2 (ROW)
- new net: D?.2 (A), K_five.2 (ROW)
- new net: D?.2 (A), K_T.2 (ROW)
- new net: D?.2 (A), K_G.2 (ROW)
- new net: D?.2 (A), K_B.2 (ROW)
- new net: D?.2 (A), K_space.2 (ROW)
- new net: D?.2 (A), K_F5.2 (ROW)
- new net: D?.2 (A), K_six.2 (ROW)
- new net: D?.2 (A), K_Y.2 (ROW)
- new net: D?.2 (A), K_H.2 (ROW)
- new net: D?.2 (A), K_N.2 (ROW)
- new net: D?.2 (A), K_F6.2 (ROW)
- new net: D?.2 (A), K_seven.2 (ROW)
- new net: D?.2 (A), K_U.2 (ROW)
- new net: D?.2 (A), K_J.2 (ROW)
- new net: D?.2 (A), K_M.2 (ROW)
- new net: D?.2 (A), K_F7.2 (ROW)
- new net: D?.2 (A), K_eight.2 (ROW)
- new net: D?.2 (A), K_I.2 (ROW)
- new net: D?.2 (A), K_K.2 (ROW)
- new net: D?.2 (A), K_comma.2 (ROW)
- new net: D?.2 (A), K_F8.2 (ROW)
- new net: D?.2 (A), K_nine.2 (ROW)
- new net: D?.2 (A), K_O.2 (ROW)
- new net: D?.2 (A), K_L.2 (ROW)
- new net: D?.2 (A), K_period.2 (ROW)
- new net: D?.2 (A), K_rightAlt.2 (ROW)
- new net: D?.2 (A), K_F9.2 (ROW)
- new net: D?.2 (A), K_zero.2 (ROW)
- new net: D?.2 (A), K_P.2 (ROW)
- new net: D?.2 (A), K_colon.2 (ROW)
- new net: D?.2 (A), K_questionMark.2 (ROW)
- new net: D?.2 (A), K_fn.2 (ROW)
- new net: D?.2 (A), K_F10.2 (ROW)
- new net: D?.2 (A), K_negative.2 (ROW)
- new net: D?.2 (A), K_openBracket.2 (ROW)
- new net: D?.2 (A), K_quote.2 (ROW)
- new net: D?.2 (A), K_F11.2 (ROW)
- new net: D?.2 (A), K_equals.2 (ROW)
- new net: D?.2 (A), K_closeBracket.2 (ROW)
- new net: D?.2 (A), K_enter.2 (ROW)
- new net: D?.2 (A), K_rightShift.2 (ROW)
- new net: D?.2 (A), K_menu.2 (ROW)
- new net: D?.2 (A), K_rightControl.2 (ROW)
- new net: D?.2 (A), K_F12.2 (ROW)
- new net: D?.2 (A), K_backspace.2 (ROW)
- new net: D?.2 (A), K_backSlash.2 (ROW)
- new net: D?.2 (A), K_left.2 (ROW)
- new net: D?.2 (A), K_printScreen.2 (ROW)
- new net: D?.2 (A), K_insert.2 (ROW)
- new net: D?.2 (A), K_delete.2 (ROW)
- new net: D?.2 (A), K_down.2 (ROW)
- new net: D?.2 (A), K_scrollLock.2 (ROW)
- new net: D?.2 (A), K_home.2 (ROW)
- new net: D?.2 (A), K_end.2 (ROW)
- new net: D?.2 (A), K_right.2 (ROW)
- new net: D?.2 (A), K_pause.2 (ROW)
- new net: D?.2 (A), K_pageUp.2 (ROW)
- new net: D?.2 (A), K_pageDown.2 (ROW)
- new net: D?.2 (A), K_up.2 (ROW)
- new net: D?.2 (A), K_numLock.2 (ROW)
- new net: D?.2 (A), K_7.2 (ROW)
- new net: D?.2 (A), K_4.2 (ROW)
- new net: D?.2 (A), K_1.2 (ROW)
- new net: D?.2 (A), K_0.2 (ROW)
- new net: D?.2 (A), K_divide.2 (ROW)
- new net: D?.2 (A), K_8.2 (ROW)
- new net: D?.2 (A), K_5.2 (ROW)
- new net: D?.2 (A), K_2.2 (ROW)
- new net: D?.2 (A), K_multiply.2 (ROW)
- new net: D?.2 (A), K_9.2 (ROW)
- new net: D?.2 (A), K_6.2 (ROW)
- new net: D?.2 (A), K_3.2 (ROW)
- new net: D?.2 (A), K_decimal.2 (ROW)
- new net: D?.2 (A), k_minus.2 (ROW)
- new net: D?.2 (A), K_tallEnter.2 (ROW)
- new net: D?.2 (A), k_plus.2 (ROW)
- new net: LED?.2 (DOUT), LED?.4 (DIN) (x7)
- new net COL0: K_ESC.1 (COL), K_capsLock.1 (COL), K_leftControl.1 (COL), K_leftShift.1 (COL), K_tab.1 (COL), K_tilde.1 (COL)
- new net COL1: K_A.1 (COL), K_Q.1 (COL), K_Z.1 (COL), K_one.1 (COL), K_windows.1 (COL)
- new net COL10: K_F9.1 (COL), K_P.1 (COL), K_colon.1 (COL), K_fn.1 (COL), K_questionMark.1 (COL), K_zero.1 (COL)
- new net COL11: K_F10.1 (COL), K_negative.1 (COL), K_openBracket.1 (COL), K_quote.1 (COL)
- new net COL12: K_F11.1 (COL), K_closeBracket.1 (COL), K_enter.1 (COL), K_equals.1 (COL), K_menu.1 (COL), K_rightShift.1 (COL)
- new net COL13: K_F12.1 (COL), K_backSlash.1 (COL), K_backspace.1 (COL), K_rightControl.1 (COL)
- new net COL14: K_delete.1 (COL), K_insert.1 (COL), K_left.1 (COL), K_printScreen.1 (COL)
- new net COL15: K_down.1 (COL), K_end.1 (COL), K_home.1 (COL), K_scrollLock.1 (COL), K_up.1 (COL)
- new net COL16: K_pageDown.1 (COL), K_pageUp.1 (COL), K_pause.1 (COL), K_right.1 (COL)
- new net COL17: K_0.1 (COL), K_1.1 (COL), K_4.1 (COL), K_7.1 (COL), K_numLock.1 (COL)
- new net COL18: K_2.1 (COL), K_5.1 (COL), K_8.1 (COL), K_divide.1 (COL)
- new net COL19: K_3.1 (COL), K_6.1 (COL), K_9.1 (COL), K_decimal.1 (COL), K_multiply.1 (COL)
- new net COL2: K_F1.1 (COL), K_S.1 (COL), K_W.1 (COL), K_X.1 (COL), K_leftAlt.1 (COL), K_two.1 (COL)
- new net COL20: K_tallEnter.1 (COL), k_minus.1 (COL), k_plus.1 (COL)
- new net COL3: K_C.1 (COL), K_D.1 (COL), K_E.1 (COL), K_F2.1 (COL), K_three.1 (COL)
- new net COL4: K_F.1 (COL), K_F3.1 (COL), K_R.1 (COL), K_V.1 (COL), K_four.1 (COL)
- new net COL5: K_B.1 (COL), K_F4.1 (COL), K_G.1 (COL), K_T.1 (COL), K_five.1 (COL), K_space.1 (COL)
- new net COL6: K_F5.1 (COL), K_H.1 (COL), K_N.1 (COL), K_Y.1 (COL), K_six.1 (COL)
- new net COL7: K_F6.1 (COL), K_J.1 (COL), K_M.1 (COL), K_U.1 (COL), K_seven.1 (COL)
- new net COL8: K_F7.1 (COL), K_I.1 (COL), K_K.1 (COL), K_comma.1 (COL), K_eight.1 (COL)
- new net COL9: K_F8.1 (COL), K_L.1 (COL), K_O.1 (COL), K_nine.1 (COL), K_period.1 (COL), K_rightAlt.1 (COL)
- new net RGBLED: LED?.4 (DIN)
- new net ROW0: D?.1 (K), D?.1 (K), D?.1 (K), D?.1 (K), D?.1 (K), D?.1 (K), D?.1 (K), D?.1 (K), D?.1 (K), D?.1 (K), D?.1 (K), D?.1 (K), D?.1 (K), D?.1 (K), D?.1 (K), D?.1 (K)
- new net ROW1: D?.1 (K), D?.1 (K), D?.1 (K), D?.1 (K), D?.1 (K), D?.1 (K), D?.1 (K), D?.1 (K), D?.1 (K), D?.1 (K), D?.1 (K), D?.1 (K), D?.1 (K), D?.1 (K), D?.1 (K), D?.1 (K), D?.1 (K), D?.1 (K), D?.1 (K), D?.1 (K), D?.1 (K)
- new net ROW2: D?.1 (K), D?.1 (K), D?.1 (K), D?.1 (K), D?.1 (K), D?.1 (K), D?.1 (K), D?.1 (K), D?.1 (K), D?.1 (K), D?.1 (K), D?.1 (K), D?.1 (K), D?.1 (K), D?.1 (K), D?.1 (K), D?.1 (K), D?.1 (K), D?.1 (K), D?.1 (K)
- new net ROW3: D?.1 (K), D?.1 (K), D?.1 (K), D?.1 (K), D?.1 (K), D?.1 (K), D?.1 (K), D?.1 (K), D?.1 (K), D?.1 (K), D?.1 (K), D?.1 (K), D?.1 (K), D?.1 (K), D?.1 (K), D?.1 (K), D?.1 (K)
- new net ROW4: D?.1 (K), D?.1 (K), D?.1 (K), D?.1 (K), D?.1 (K), D?.1 (K), D?.1 (K), D?.1 (K), D?.1 (K), D?.1 (K), D?.1 (K), D?.1 (K), D?.1 (K), D?.1 (K), D?.1 (K), D?.1 (K)
- new net ROW5: D?.1 (K), D?.1 (K), D?.1 (K), D?.1 (K), D?.1 (K), D?.1 (K), D?.1 (K), D?.1 (K), D?.1 (K), D?.1 (K), D?.1 (K), D?.1 (K), D?.1 (K), D?.1 (K)
- no-connect marks 0 -> 1
Other:
- moved on the sheet: C?, F?, R?, SW?, U?, USB?, Y?
