File: DOMAIN-1/DOMAIN-1.sch (KiCad schematic (older format))
At the start: 235 parts

Commit message: Finished PCB matrix
Parts:
- added J1: Conn_02x10_Odd_Even, Connector_IDC:IDC-Header_2x10_P2.54mm_Horizontal, symbol Connector_Generic:Conn_02x10_Odd_Even
- added J2: AVR-ISP-6, random-keyboard-parts:Reset_Pretty-Mask, symbol Connector:AVR-ISP-6
- C1, C2, C3, C4, C5, C6, C7: renamed from C?; footprint (none) -> Capacitor_SMD:C_0603_1608Metric
- D1, D10, D100, D101, D102, D103, D104, D11, D12, D13, D14, D15, D16, D17, D18, D19, D2, D20, D21, D22, D23, D24, D25, D26, D27, D28, D29, D3, D30, D31, D32, D33, D34, D35, D36, D37, D38, D39, D4, D40, D41, D42, D43, D44, D45, D46, D47, D48, D49, D5, D50, D51, D52, D53, D54, D55, D56, D57, D58, D59, D6, D60, D61, D62, D63, D64, D65, D66, D67, D68, D69, D7, D70, D71, D72, D73, D74, D75, D76, D77, D78, D79, D8, D80, D81, D82, D83, D84, D85, D86, D87, D88, D89, D9, D90, D91, D92, D93, D94, D95, D96, D97, D98, D99: renamed from D?; footprint (none) -> Diode_SMD:D_SOD-123
- F1: renamed from F?; value Polyfuse_Small -> 500mA; footprint (none) -> Fuse:Fuse_1206_3216Metric
- K_0: footprint (none) -> MX_Only:MXOnly-2U-Hotswap
- K_1, K_2, K_3, K_4, K_5, K_6, K_7, K_8, K_9, K_F1, K_F10, K_F11, K_F12, K_F2, K_F3, K_F4, K_F5, K_F6, K_F7, K_F8, K_F9: footprint (none) -> MX_Only:MXOnly-1U-Hotswap
- K_A1: renamed from K_A; footprint (none) -> MX_Only:MXOnly-1U-Hotswap
- K_B1: renamed from K_B; footprint (none) -> MX_Only:MXOnly-1U-Hotswap
- K_C1: renamed from K_C; footprint (none) -> MX_Only:MXOnly-1U-Hotswap
- K_D1: renamed from K_D; footprint (none) -> MX_Only:MXOnly-1U-Hotswap
- K_E1: renamed from K_E; footprint (none) -> MX_Only:MXOnly-1U-Hotswap
- K_ESC1: renamed from K_ESC; footprint (none) -> MX_Only:MXOnly-1U-Hotswap
- K_F13: renamed from K_F; footprint (none) -> MX_Only:MXOnly-1U-Hotswap
- K_G1: renamed from K_G; footprint (none) -> MX_Only:MXOnly-1U-Hotswap
- K_H1: renamed from K_H; footprint (none) -> MX_Only:MXOnly-1U-Hotswap
- K_I1: renamed from K_I; footprint (none) -> MX_Only:MXOnly-1U-Hotswap
- K_J1: renamed from K_J; footprint (none) -> MX_Only:MXOnly-1U-Hotswap
- K_K1: renamed from K_K; footprint (none) -> MX_Only:MXOnly-1U-Hotswap
- K_L1: renamed from K_L; footprint (none) -> MX_Only:MXOnly-1U-Hotswap
- K_M1: renamed from K_M; footprint (none) -> MX_Only:MXOnly-1U-Hotswap
- K_N1: renamed from K_N; footprint (none) -> MX_Only:MXOnly-1U-Hotswap
- K_O1: renamed from K_O; footprint (none) -> MX_Only:MXOnly-1U-Hotswap
- K_P1: renamed from K_P; footprint (none) -> MX_Only:MXOnly-1U-Hotswap
- K_Q1: renamed from K_Q; footprint (none) -> MX_Only:MXOnly-1U-Hotswap
- K_R1: renamed from K_R; footprint (none) -> MX_Only:MXOnly-1U-Hotswap
- K_S1: renamed from K_S; footprint (none) -> MX_Only:MXOnly-1U-Hotswap
- K_T1: renamed from K_T; footprint (none) -> MX_Only:MXOnly-1U-Hotswap
- K_U1: renamed from K_U; footprint (none) -> MX_Only:MXOnly-1U-Hotswap
- K_V1: renamed from K_V; footprint (none) -> MX_Only:MXOnly-1U-Hotswap
- K_W1: renamed from K_W; footprint (none) -> MX_Only:MXOnly-1U-Hotswap
- K_X1: renamed from K_X; footprint (none) -> MX_Only:MXOnly-1U-Hotswap
- K_Y1: renamed from K_Y; footprint (none) -> MX_Only:MXOnly-1U-Hotswap
- K_Z1: renamed from K_Z; footprint (none) -> MX_Only:MXOnly-1U-Hotswap
- K_backSlash1: renamed from K_backSlash; footprint (none) -> MX_Only:MXOnly-1.5U-Hotswap
- K_backspace1: renamed from K_backspace; footprint (none) -> MX_Only:MXOnly-2U-Hotswap
- K_capsLock1: renamed from K_capsLock; footprint (none) -> MX_Only:MXOnly-1.75U-Hotswap
- K_closeBracket1: renamed from K_closeBracket; footprint (none) -> MX_Only:MXOnly-1U-Hotswap
- K_colon1: renamed from K_colon; footprint (none) -> MX_Only:MXOnly-1U-Hotswap
- K_comma1: renamed from K_comma; footprint (none) -> MX_Only:MXOnly-1U-Hotswap
- K_decimal1: renamed from K_decimal; footprint (none) -> MX_Only:MXOnly-1U-Hotswap
- K_delete1: renamed from K_delete; footprint (none) -> MX_Only:MXOnly-1U-Hotswap
- K_divide1: renamed from K_divide; footprint (none) -> MX_Only:MXOnly-1U-Hotswap
- K_down1: renamed from K_down; footprint (none) -> MX_Only:MXOnly-1U-Hotswap
- K_eight1: renamed from K_eight; footprint (none) -> MX_Only:MXOnly-1U-Hotswap
- K_end1: renamed from K_end; footprint (none) -> MX_Only:MXOnly-1U-Hotswap
- K_enter1: renamed from K_enter; footprint (none) -> MX_Only:MXOnly-2.25U-Hotswap
- K_equals1: renamed from K_equals; footprint (none) -> MX_Only:MXOnly-1U-Hotswap
- K_five1: renamed from K_five; footprint (none) -> MX_Only:MXOnly-1U-Hotswap
- K_fn1: renamed from K_fn; footprint (none) -> MX_Only:MXOnly-1.25U-Hotswap
- K_four1: renamed from K_four; footprint (none) -> MX_Only:MXOnly-1U-Hotswap
- K_home1: renamed from K_home; footprint (none) -> MX_Only:MXOnly-1U-Hotswap
- K_insert1: renamed from K_insert; footprint (none) -> MX_Only:MXOnly-1U-Hotswap
- K_left1: renamed from K_left; footprint (none) -> MX_Only:MXOnly-1U-Hotswap
- K_leftAlt1: renamed from K_leftAlt; footprint (none) -> MX_Only:MXOnly-1.25U-Hotswap
- K_leftControl1: renamed from K_leftControl; footprint (none) -> MX_Only:MXOnly-1.25U-Hotswap
- K_leftShift1: renamed from K_leftShift; footprint (none) -> MX_Only:MXOnly-2.25U-Hotswap
- K_menu1: renamed from K_menu; footprint (none) -> MX_Only:MXOnly-1.25U-Hotswap
- K_multiply1: renamed from K_multiply; footprint (none) -> MX_Only:MXOnly-1U-Hotswap
- K_negative1: renamed from K_negative; footprint (none) -> MX_Only:MXOnly-1U-Hotswap
- K_nine1: renamed from K_nine; footprint (none) -> MX_Only:MXOnly-1U-Hotswap
- K_numLock1: renamed from K_numLock; footprint (none) -> MX_Only:MXOnly-1U-Hotswap
- K_one1: renamed from K_one; footprint (none) -> MX_Only:MXOnly-1U-Hotswap
- K_openBracket1: renamed from K_openBracket; footprint (none) -> MX_Only:MXOnly-1U-Hotswap
- K_pageDown1: renamed from K_pageDown; footprint (none) -> MX_Only:MXOnly-1U-Hotswap
- K_pageUp1: renamed from K_pageUp; footprint (none) -> MX_Only:MXOnly-1U-Hotswap
- K_pause1: renamed from K_pause; footprint (none) -> MX_Only:MXOnly-1U-Hotswap
- K_period1: renamed from K_period; footprint (none) -> MX_Only:MXOnly-1U-Hotswap
- K_printScreen1: renamed from K_printScreen; footprint (none) -> MX_Only:MXOnly-1U-Hotswap
- K_questionMark1: renamed from K_questionMark; footprint (none) -> MX_Only:MXOnly-1U-Hotswap
- K_quote1: renamed from K_quote; footprint (none) -> MX_Only:MXOnly-1U-Hotswap
- K_right1: renamed from K_right; footprint (none) -> MX_Only:MXOnly-1U-Hotswap
- K_rightAlt1: renamed from K_rightAlt; footprint (none) -> MX_Only:MXOnly-1.25U-Hotswap
- K_rightControl1: renamed from K_rightControl; footprint (none) -> MX_Only:MXOnly-1.25U-Hotswap
- K_rightShift1: renamed from K_rightShift; footprint (none) -> MX_Only:MXOnly-2.75U-Hotswap
- K_scrollLock1: renamed from K_scrollLock; footprint (none) -> MX_Only:MXOnly-1U-Hotswap
- K_seven1: renamed from K_seven; footprint (none) -> MX_Only:MXOnly-1U-Hotswap
- K_six1: renamed from K_six; footprint (none) -> MX_Only:MXOnly-1U-Hotswap
- K_space1: renamed from K_space; footprint (none) -> MX_Only:MXOnly-6.25U-Hotswap
- K_tab1: renamed from K_tab; footprint (none) -> MX_Only:MXOnly-1.5U-Hotswap
- K_tallEnter1: renamed from K_tallEnter; footprint (none) -> MX_2U_Hotswap_Vertical:MX-2U-Hotswap-Vertical
- K_three1: renamed from K_three; footprint (none) -> MX_Only:MXOnly-1U-Hotswap
- K_tilde1: renamed from K_tilde; footprint (none) -> MX_Only:MXOnly-1U-Hotswap
- K_two1: renamed from K_two; footprint (none) -> MX_Only:MXOnly-1U-Hotswap
- K_up1: renamed from K_up; footprint (none) -> MX_Only:MXOnly-1U-Hotswap
- K_windows1: renamed from K_windows; footprint (none) -> MX_Only:MXOnly-1.25U-Hotswap
- K_zero1: renamed from K_zero; footprint (none) -> MX_Only:MXOnly-1U-Hotswap
- LED1, LED2, LED3, LED4, LED5, LED6, LED7, LED8: renamed from LED?; footprint (none) -> WS2812B:WS2812B
- R1, R2, R3, R4, R5, R6: renamed from R?; footprint (none) -> Resistor_SMD:R_0805_2012Metric
- SW1: renamed from SW?; footprint (none) -> random-keyboard-parts:SKQG-1155865
- U2: renamed from U?; footprint (none) -> random-keyboard-parts:SOT143B
- USB1: renamed from USB?; footprint (none) -> Type-C:HRO-TYPE-C-31-M-12-Assembly
- Y1: renamed from Y?; footprint (none) -> Crystal:Crystal_SMD_3225-4Pin_3.2x2.5mm
- k_minus1: renamed from k_minus; footprint (none) -> MX_Only:MXOnly-1U-Hotswap
- k_plus1: renamed from k_plus; footprint (none) -> MX_2U_Hotswap_Vertical:MX-2U-Hotswap-Vertical
- gave numbers to parts that had none: 1
Connections:
- net +5V: now also J1.17 (Pin_17), J2.2 (VCC)
- net COL0: now also U1.51 (PA0)
- net COL1: now also U1.50 (PA1)
- net COL10: now also U1.16 (PB6), J1.3 (Pin_3)
- net COL11: now also U1.17 (PB7), J1.2 (Pin_2)
- net COL12: now also U1.35 (PC0), J1.4 (Pin_4)
- net COL13: now also U1.36 (PC1), J1.6 (Pin_6)
- net COL14: now also U1.37 (PC2), J1.8 (Pin_8)
- net COL15: now also U1.38 (PC3), J1.10 (Pin_10)
- net COL16: now also U1.39 (PC4), J1.12 (Pin_12)
- net COL17: now also U1.40 (PC5), J1.14 (Pin_14)
- net COL18: now also U1.41 (PC6), J1.16 (Pin_16)
- net COL19: now also U1.42 (PC7), J1.18 (Pin_18)
- net COL2: now also U1.49 (PA2)
- net COL20: now also U1.25 (PD0), J1.20 (Pin_20)
- net COL3: now also U1.48 (PA3)
- net COL4: now also U1.47 (PA4)
- net COL5: now also U1.46 (PA5)
- net COL6: now also U1.45 (PA6)
- net COL7: now also U1.44 (PA7)
- net COL8: now also U1.10 (PB0)
- net COL9: now also U1.14 (PB4), J1.5 (Pin_5)
- net GND: now also J1.19 (Pin_19), J2.6 (GND)
- net RGBLED: now also U1.15 (PB5)
- net ROW0: now also U1.26 (PD1)
- net ROW1: now also U1.27 (PD2)
- net ROW2: now also U1.28 (PD3)
- net ROW3: now also U1.29 (PD4)
- net ROW4: now also U1.30 (PD5)
- net ROW5: now also U1.31 (PD6)
- net SCK: now reaches U1.11 (PB1)
- net SCK: now also J2.3 (SCK)
- net MOSI: now reaches U1.12 (PB2)
- net MOSI: now also J2.4 (MOSI)
- net MISO: now reaches U1.13 (PB3)
- net MISO: now also J2.1 (MISO)
- net RESET: now reaches R1.2, SW1.2, U1.20 (~RESET)
- net RESET: now also J2.5 (~RST)
- net ROW6: now reaches U1.32 (PD7)
- net ROW6: now also J1.7 (Pin_7)
- net ROW7: now reaches U1.54 (PF7)
- net ROW7: now also J1.9 (Pin_9)
- net RGBLED_toUpperBoard: now reaches LED8.2 (DOUT)
- net RGBLED_toUpperBoard: now also J1.1 (Pin_1)
- no-connect marks 1 -> 0
Other:
- moved on the sheet: C1, C2, C3, C4, C5, C6, C7, F1, LED1, LED2, LED3, LED4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

Commit message: Finished PCB layout
Parts:
- added C10, C11, C12, C13, C14, C15, C8, C9: 0.1uF, Capacitor_SMD:C_0603_1608Metric, symbol Device:C_Small
- renumbered LED3 to LED2, LED5 to LED3, LED7 to LED4, LED2 to LED5, LED4 to LED6, LED6 to LED7
Connections:
- net +5V: now also C10.1, C11.1, C12.1, C13.1, C14.1, C15.1, C8.1, C9.1
- net GND: now also C10.2, C11.2, C12.2, C13.2, C14.2, C15.2, C8.2, C9.2
Changed lines of the file:
@@
 $EndComp
 $Comp
-L ws2812b:WS2812B LED3
+L ws2812b:WS2812B LED2
 U 1 1 623D24D5
 P 4650 8200
-F 0 "LED3" H 4650 8687 60  0000 C CNN
+F 0 "LED2" H 4650 8687 60  0000 C CNN
 F 1 "WS2812B" H 4650 8581 60  0000 C CNN
 F 2 "WS2812B:WS2812B" V 4600 8200 60  0001 C CNN
@@
 $EndComp
 $Comp
-L ws2812b:WS2812B LED5
+L ws2812b:WS2812B LED3
 U 1 1 623E82C4
 P 4650 9150
-F 0 "LED5" H 4650 9637 60  0000 C CNN
+F 0 "LED3" H 4650 9637 60  0000 C CNN
 F 1 "WS2812B" H 4650 9531 60  0000 C CNN
 F 2 "WS2812B:WS2812B" V 4600 9150 60  0001 C CNN
@@
 $EndComp
 $Comp
-L ws2812b:WS2812B LED7
+L ws2812b:WS2812B LED4
 U 1 1 623FDDAE
 P 4650 10100
-F 0 "LED7" H 4650 10587 60  0000 C CNN
+F 0 "LED4" H 4650 10587 60  0000 C CNN
 F 1 "WS2812B" H 4650 10481 60  0000 C CNN
 F 2 "WS2812B:WS2812B" V 4600 10100 60  0001 C CNN
@@
 $EndComp
 $Comp
-L ws2812b:WS2812B LED2
+L ws2812b:WS2812B LED5
 U 1 1 624309B6
 P 6300 7300
-F 0 "LED2" H 6300 7787 60  0000 C CNN
+F 0 "LED5" H 6300 7787 60  0000 C CNN
 F 1 "WS2812B" H 6300 7681 60  0000 C CNN
 F 2 "WS2812B:WS2812B" V 6250 7300 60  0001 C CNN
@@
 $EndComp
 $Comp
-L ws2812b:WS2812B LED4
+L ws2812b:WS2812B LED6
 U 1 1 624309BC
 P 6300 8200
-F 0 "LED4" H 6300 8687 60  0000 C CNN
+F 0 "LED6" H 6300 8687 60  0000 C CNN
 F 1 "WS2812B" H 6300 8581 60  0000 C CNN
 F 2 "WS2812B:WS2812B" V 6250 8200 60  0001 C CNN
@@
 $EndComp
 $Comp
-L ws2812b:WS2812B LED6
+L ws2812b:WS2812B LED7
 U 1 1 624309C2
 P 6300 9150
-F 0 "LED6" H 6300 9637 60  0000 C CNN
+F 0 "LED7" H 6300 9637 60  0000 C CNN
 F 1 "WS2812B" H 6300 9531 60  0000 C CNN
 F 2 "WS2812B:WS2812B" V 6250 9150 60  0001 C CNN
@@
 Text GLabel 2250 10550 0    50   Input ~ 0
 ROW7
+$Comp
+L Device:C_Small C8
+U 1 1 621AC69C
+P 13000 6950
+F 0 "C8" H 13092 6996 50  0000 L CNN
+F 1 "0.1uF" H 13092 6905 50  0000 L CNN
+F 2 "Capacitor_SMD:C_0603_1608Metric" H 13000 6950 50  0001 C CNN
+F 3 "~" H 13000 6950 50  0001 C CNN
+	1    13000 6950
+	1    0    0    -1
+$EndComp
+$Comp
+L Device:C_Small C9
+U 1 1 621AE816
+P 13550 6950
+F 0 "C9" H 13642 6996 50  0000 L CNN
+F 1 "0.1uF" H 13642 6905 50  0000 L CNN
+F 2 "Capacitor_SMD:C_0603_1608Metric" H 13550 6950 50  0001 C CNN
+F 3 "~" H 13550 6950 50  0001 C CNN
+	1    13550 6950
+	1    0    0    -1
+$EndComp
+$Comp
+L Device:C_Small C10
+U 1 1 621D0AD8
+P 14100 6950
+F 0 "C10" H 14192 6996 50  0000 L CNN
+F 1 "0.1uF" H 14192 6905 50  0000 L CNN
+F 2 "Capacitor_SMD:C_0603_1608Metric" H 14100 6950 50  0001 C CNN
+F 3 "~" H 14100 6950 50  0001 C CNN
+	1    14100 6950
+	1    0    0    -1
+$EndComp
+$Comp
+L Device:C_Small C11
+U 1 1 621D0ADE
+P 14650 6950
+F 0 "C11" H 14742 6996 50  0000 L CNN
+F 1 "0.1uF" H 14742 6905 50  0000 L CNN
+F 2 "Capacitor_SMD:C_0603_1608Metric" H 14650 6950 50  0001 C CNN
+F 3 "~" H 14650 6950 50  0001 C CNN
+	1    14650 6950
+	1    0    0    -1
+$EndComp
+$Comp
+L Device:C_Small C12
+U 1 1 621F3500
+P 13000 7350
+F 0 "C12" H 13092 7396 50  0000 L CNN
+F 1 "0.1uF" H 13092 7305 50  0000 L CNN
+F 2 "Capacitor_SMD:C_0603_1608Metric" H 13000 7350 50  0001 C CNN
+F 3 "~" H 13000 7350 50  0001 C CNN
+	1    13000 7350
+	1    0    0    -1
+$EndComp
+$Comp
+L Device:C_Small C13
+U 1 1 621F3506
+P 13550 7350
+F 0 "C13" H 13642 7396 50  0000 L CNN
+F 1 "0.1uF" H 13642 7305 50  0000 L CNN
+F 2 "Capacitor_SMD:C_0603_1608Metric" H 13550 7350 50  0001 C CNN
+F 3 "~" H 13550 7350 50  0001 C CNN
+	1    13550 7350
+	1    0    0    -1
+$EndComp
+$Comp
+L Device:C_Small C14
+U 1 1 621F350C
+P 14100 7350
+F 0 "C14" H 14192 7396 50  0000 L CNN
+F 1 "0.1uF" H 14192 7305 50  0000 L CNN
+F 2 "Capacitor_SMD:C_0603_1608Metric" H 14100 7350 50  0001 C CNN
+F 3 "~" H 14100 7350 50  0001 C CNN
+	1    14100 7350
+	1    0    0    -1
+$EndComp
+$Comp
+L Device:C_Small C15
+U 1 1 621F3512
+P 14650 7350
+F 0 "C15" H 14742 7396 50  0000 L CNN
+F 1 "0.1uF" H 14742 7305 50  0000 L CNN
+F 2 "Capacitor_SMD:C_0603_1608Metric" H 14650 7350 50  0001 C CNN
+F 3 "~" H 14650 7350 50  0001 C CNN
+	1    14650 7350
+	1    0    0    -1
+$EndComp
+Wire Wire Line
+	13000 6850 13550 6850
+Connection ~ 13550 6850
+Wire Wire Line
+	13550 6850 14100 6850
+Connection ~ 14100 6850
+Wire Wire Line
+	14100 6850 14650 6850
+Wire Wire Line
+	14650 7250 14100 7250
+Wire Wire Line
+	12650 7250 12650 6850
+Connection ~ 13000 7250
+Wire Wire Line
+	13000 7250 12650 7250
+Connection ~ 13550 7250
+Wire Wire Line
+	13550 7250 13000 7250
+Connection ~ 14100 7250
+Wire Wire Line
+	14100 7250 13550 7250
+Wire Wire Line
+	13000 6850 12650 6850
+Connection ~ 13000 6850
+Connection ~ 12650 6850
+Wire Wire Line
+	12650 6850 12650 6750
+$Comp
+L power:+5V #PWR0123
+U 1 1 6227F464
+P 12650 6750
+F 0 "#PWR0123" H 12650 6600 50  0001 C CNN
+F 1 "+5V" H 12665 6923 50  0000 C CNN
+F 2 "" H 12650 6750 50  0001 C CNN
+F 3 "" H 12650 6750 50  0001 C CNN
+	1    12650 6750
+	1    0    0    -1
+$EndComp
+Wire Wire Line
+	13000 7450 13550 7450
+Wire Wire Line
+	15300 7450 15300 7550
+Connection ~ 13550 7450
+Wire Wire Line
+	13550 7450 14100 7450
+Connection ~ 14100 7450
+Wire Wire Line
+	14100 7450 14650 7450
+Connection ~ 14650 7450
+Wire Wire Line
+	14650 7450 15300 7450
+Wire Wire Line
+	13000 7050 13550 7050
+Wire Wire Line
+	15300 7050 15300 7450
+Connection ~ 13550 7050
+Wire Wire Line
+	13550 7050 14100 7050
+Connection ~ 14100 7050
+Wire Wire Line
+	14100 7050 14650 7050
+Connection ~ 14650 7050
+Wire Wire Line
+	14650 7050 15300 7050
+Connection ~ 15300 7450
+$Comp
+L power:GND #PWR0124
+U 1 1 622CA081
+P 15300 7550
+F 0 "#PWR0124" H 15300 7300 50  0001 C CNN
+F 1 "GND" H 15305 7377 50  0000 C CNN
+F 2 "" H 15300 7550 50  0001 C CNN
+F 3 "" H 15300 7550 50  0001 C CNN
+	1    15300 7550
+	1    0    0    -1
+$EndComp
 $EndSCHEMATC
