File: DOMAIN-1/DOMAIN-1.kicad_pcb (KiCad board)
At the start: 2 copper layers, 237 parts, among them J1 Conn_02x10_Odd_Even, J2 AVR-ISP-6, SW1 SW_Push, U1 AT90USB1286-AU, U2 PRTR5V0U2X, Y1 Crystal_GND24_Small

Commit message: Finished PCB layout
Parts:
- added C10: 0.1uF, Capacitor_SMD:C_0603_1608Metric, B.Cu at (85.6, 214.2)
- added C11: 0.1uF, Capacitor_SMD:C_0603_1608Metric, B.Cu at (85.3, 239.5)
- added C12: 0.1uF, Capacitor_SMD:C_0603_1608Metric, B.Cu at (513.8, 256.7)
- added C13: 0.1uF, Capacitor_SMD:C_0603_1608Metric, B.Cu at (514.4, 223.0)
- added C14: 0.1uF, Capacitor_SMD:C_0603_1608Metric, B.Cu at (513.8, 185.7)
- added C15: 0.1uF, Capacitor_SMD:C_0603_1608Metric, B.Cu at (514.2, 157.5)
- added C8: 0.1uF, Capacitor_SMD:C_0603_1608Metric, B.Cu at (92.1, 166.0)
- added C9: 0.1uF, Capacitor_SMD:C_0603_1608Metric, B.Cu at (85.1, 187.2)
- C1, C2, C3, C4, C5, C6, C7, D1, D10, D100, D101, D102, D103, D104, D11, D12, D13, D14, D15, D16, D17, D18, D19, D2, D20, D21, D22, D23, D24, D25, D26, D27, D28, D29, D3, D30, D31, D32, D33, D34, D35, D36, D37, D38, D39, D4, D40, D41, D42, D43, D44, D45, D46, D47, D48, D49, D5, D50, D51, D52, D53, D54, D55, D56, D57, D58, D59, D6, D60, D61, D62, D63, D64, D65, D66, D67, D68, D69, D7, D70, D71, D72, D73, D74, D75, D76, D77, D78, D79, D8, D80, D81, D82, D83, D84, D85, D86, D87, D88, D89, D9, D90, D91, D92, D93, D94, D95, D96, D97, D98, D99, F1, J1, J2, LED1, LED8, R1, R2, R3, R4, R5, R6, SW1, U1, U2, USB1, Y1: moved to B.Cu
- LED2: renamed from LED3; moved to B.Cu
- LED3: renamed from LED5; moved to B.Cu
- LED4: renamed from LED7; moved to B.Cu
- LED5: renamed from LED2; moved to B.Cu
- LED6: renamed from LED4; moved to B.Cu
- LED7: renamed from LED6; moved to B.Cu
- moved D103 705.5 mm to (486.7, 263.4), turned to 90 degrees
- moved J1 665.6 mm to (479.6, 153.5), turned to 90 degrees
- moved D102 648.4 mm to (458.1, 263.4), turned to 90 degrees
- moved D101 620.9 mm to (424.8, 263.4), turned to 90 degrees
- moved D100 607.7 mm to (405.8, 263.4), turned to 90 degrees
- moved D99 594.5 mm to (386.7, 263.4), turned to 90 degrees
- moved D74 586.0 mm to (505.7, 215.8), turned to 90 degrees
- moved C7 581.9 mm to (386.3, 213.6), turned to 90 degrees
- moved D90 579.4 mm to (486.7, 244.3), turned to 90 degrees
- moved C5 575.0 mm to (390.1, 221.1), turned to 270 degrees
- moved D98 574.0 mm to (360.4, 263.4), turned to 90 degrees
- moved C1 567.9 mm to (371.0, 241.8), turned to 270 degrees
- moved C4 566.6 mm to (382.8, 236.2), turned to 180 degrees
- moved R4 563.9 mm to (365.0, 220.9), turned to 90 degrees
- moved C6 561.5 mm to (373.8, 213.0)
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Routing:
- net ROW5: track 0.00 -> 411.1 mm
- net ROW1: track 0.00 -> 409.6 mm
- net COL2: track 0.00 -> 379.7 mm, vias 0 -> 6
- net COL1: track 0.00 -> 370.7 mm, vias 0 -> 5
- net COL3: track 0.00 -> 333.8 mm, vias 0 -> 5
- net ROW2: track 0.00 -> 333.4 mm
- net ROW4: track 0.00 -> 319.0 mm
- net COL5: track 0.00 -> 318.6 mm, vias 0 -> 6
- net COL4: track 0.00 -> 315.5 mm, vias 0 -> 5
- net ROW3: track 0.00 -> 309.2 mm
- net ROW0: track 0.00 -> 301.1 mm
- net COL0: track 0.00 -> 283.9 mm
- net COL6: track 0.00 -> 279.3 mm, vias 0 -> 5
- net RGBLED: track 0.00 -> 278.9 mm
- net COL7: track 0.00 -> 261.2 mm, vias 0 -> 5
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Other:
- board outline added: 436.9 x 123.8 mm
- net class Power added: clearance 0.2, trace_width 0.381, via_dia 0.8, via_drill 0.4

Commit message: Finished LED placement
Parts:
- moved SW1 12.7 mm to (415.7, 223.9)
- moved R1 12.7 mm to (408.3, 223.9)
- moved C3 11.1 mm to (398.4, 217.7)
- moved C5 11.1 mm to (400.7, 217.7)
- moved F1 9.68 mm to (281.9, 157.3)
- moved C11 8.82 mm to (80.9, 247.1)
- moved LED4 8.49 mm to (80.5, 254.4)
- moved LED1 8.26 mm to (80.5, 160.7), turned to 0 degrees
- moved LED3 5.18 mm to (80.5, 223.1)
- moved C10 5.02 mm to (80.8, 215.6)
- moved R5 4.94 mm to (281.8, 151.6)
- moved C9 4.84 mm to (80.6, 185.3)
- moved LED2 4.62 mm to (80.5, 191.9), turned to 180 degrees
- moved R2 4.58 mm to (284.9, 155.7)
- moved R3 4.45 mm to (287.7, 155.7)
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Connections:
- R5 pad 1: Net-(R3-Pad2) -> GND
- R6 pad 1: Net-(R3-Pad2) -> GND
- U1 pad 10: COL8 -> Net-(U1-Pad10)
- U1 pad 14: COL9 -> ROW3
- U1 pad 15: RGBLED -> COL16
- U1 pad 16: COL10 -> ROW2
- U1 pad 17: COL11 -> ROW1
- U1 pad 25: COL20 -> COL14
- U1 pad 26: ROW0 -> ROW5
- U1 pad 27: ROW1 -> ROW4
- U1 pad 28: ROW2 -> COL13
- U1 pad 29: ROW3 -> COL12
- U1 pad 30: ROW4 -> COL11
- U1 pad 31: ROW5 -> COL10
- U1 pad 32: ROW6 -> COL9
- U1 pad 33: Net-(U1-Pad33) -> COL8
- U1 pad 34: Net-(U1-Pad34) -> COL7
- U1 pad 35: COL12 -> COL6
- U1 pad 36: COL13 -> COL5
- U1 pad 37: COL14 -> COL4
- U1 pad 38: COL15 -> COL3
- U1 pad 39: COL16 -> COL2
- U1 pad 40: COL17 -> COL1
- U1 pad 41: COL18 -> COL0
- U1 pad 42: COL19 -> RGBLED
- U1 pad 44: COL7 -> COL19
- U1 pad 45: COL6 -> ROW6
- U1 pad 46: COL5 -> COL18
- U1 pad 47: COL4 -> Net-(U1-Pad47)
- U1 pad 48: COL3 -> ROW0
- U1 pad 49: COL2 -> COL20
- U1 pad 50: COL1 -> COL17
- U1 pad 51: COL0 -> COL15
- U2 pad 1: Net-(R3-Pad2) -> GND
Routing:
- net GND: track 0.00 -> 565.5 mm, vias 0 -> 3
- net +5V: track 0.00 -> 484.0 mm, vias 0 -> 6
- net Net-(LED4-Pad2): track 0.00 -> 467.3 mm
- net COL0: track 283.9 -> 474.2 mm, vias 0 -> 6
- net COL11: track 163.1 -> 351.7 mm
- net COL12: track 198.8 -> 370.0 mm
- net COL13: track 156.1 -> 309.0 mm
- net ROW4: track 319.0 -> 416.6 mm
- net COL14: track 50.6 -> 137.4 mm, vias 3 -> 5
- net COL15: track 70.6 -> 152.9 mm
- net RGBLED: track 278.9 -> 351.8 mm
- net COL20: track 73.0 -> 144.9 mm
- net COL9: track 244.9 -> 316.4 mm
- net COL10: track 230.7 -> 300.2 mm
- net COL8: track 241.4 -> 305.8 mm
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- added copper zone on B.Cu, net GND
Other:
- board size 436.9 x 123.8 mm -> 441.8 x 129.4 mm

Commit message: Finished mainboard
Parts:
- moved C1 3.11 mm to (376.0, 238.9)
- moved C2 3.11 mm to (386.0, 238.9)
- moved Y1 3.11 mm to (380.9, 238.9)
- moved C4 3.06 mm to (386.8, 235.1)
- moved C5 2.54 mm to (403.2, 217.7)
- moved C6 2.43 mm to (374.4, 212.9)
- moved C7 1.89 mm to (389.6, 215.6), turned to 180 degrees
- moved R6 0.52 mm to (290.2, 152.7)
- moved R2 0.28 mm to (285.1, 155.8)
- moved R3 0.28 mm to (287.9, 155.8)
Connections:
- J1 pad 1: RGBLED_toUpperBoard -> +5V
- J1 pad 10: COL15 -> COL14
- J1 pad 12: COL16 -> COL15
- J1 pad 13: Net-(J1-Pad13) -> ROW6
- J1 pad 14: COL17 -> COL16
- J1 pad 15: Net-(J1-Pad15) -> ROW7
- J1 pad 16: COL18 -> COL10
- J1 pad 17: +5V -> Net-(J1-Pad17)
- J1 pad 18: COL19 -> Net-(J1-Pad18)
- J1 pad 2: COL11 -> RGBLED_toUpperBoard
- J1 pad 20: COL20 -> COL9
- J1 pad 3: COL10 -> COL20
- J1 pad 4: COL12 -> COL11
- J1 pad 5: COL9 -> COL19
- J1 pad 6: COL13 -> COL12
- J1 pad 7: ROW6 -> COL18
- J1 pad 8: COL14 -> COL13
- J1 pad 9: ROW7 -> COL17
- U1 pad 10: Net-(U1-Pad10) -> ROW7
- U1 pad 14: ROW3 -> ROW6
- U1 pad 15: COL16 -> COL20
- U1 pad 16: ROW2 -> COL19
- U1 pad 17: ROW1 -> COL18
- U1 pad 18: Net-(U1-Pad18) -> COL17
- U1 pad 19: Net-(U1-Pad19) -> ROW3
- U1 pad 44: COL19 -> Net-(U1-Pad44)
- U1 pad 45: ROW6 -> Net-(U1-Pad45)
- U1 pad 46: COL18 -> Net-(U1-Pad46)
- U1 pad 48: ROW0 -> Net-(U1-Pad48)
- U1 pad 49: COL20 -> Net-(U1-Pad49)
- U1 pad 50: COL17 -> Net-(U1-Pad50)
- U1 pad 51: COL15 -> Net-(U1-Pad51)
- U1 pad 54: ROW7 -> ROW2
- U1 pad 55: Net-(U1-Pad55) -> ROW1
- U1 pad 56: Net-(U1-Pad56) -> COL16
- U1 pad 57: Net-(U1-Pad57) -> COL15
- U1 pad 58: Net-(U1-Pad58) -> ROW0
Routing:
- net GND: track 565.5 -> 922.1 mm, vias 3 -> 5
- net +5V: track 484.0 -> 790.4 mm, vias 6 -> 8
- net D+: track 5.38 -> 241.1 mm
- net D-: track 4.82 -> 240.3 mm
- net COL9: track 316.4 -> 520.2 mm, vias 6 -> 8
- net COL10: track 300.2 -> 479.0 mm, vias 6 -> 7
- net COL16: track 92.9 -> 269.2 mm, vias 3 -> 4
- net COL15: track 152.9 -> 309.8 mm, vias 5 -> 7
- net ROW7: track 0.00 -> 141.9 mm, vias 0 -> 2
- net ROW6: track 0.00 -> 141.7 mm, vias 0 -> 2
- net ROW0: track 301.1 -> 436.7 mm, vias 0 -> 4
- net ROW3: track 309.2 -> 432.3 mm, vias 0 -> 2
- net COL20: track 144.9 -> 262.1 mm, vias 3 -> 5
- net COL17: track 94.2 -> 207.6 mm
- net COL18: track 96.4 -> 205.8 mm
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
Commit message: Generated gerber files
Parts:
- moved J1 5.08 mm to (479.6, 158.6)
Routing:
- net ROW2: track 417.3 -> 439.1 mm, vias 3 -> 4
- net +5V: track 790.4 -> 811.7 mm
- net COL20: track 262.1 -> 257.0 mm
- net COL19: track 244.9 -> 239.8 mm
- net COL18: track 205.8 -> 200.7 mm
- net COL17: track 207.6 -> 202.5 mm
- net ROW7: track 141.9 -> 137.8 mm
- net ROW6: track 141.7 -> 137.6 mm
- net Net-(R3-Pad2): track 8.32 -> 11.7 mm
- net RGBLED_toUpperBoard: track 42.4 -> 44.6 mm
- net COL9: track 520.2 -> 518.1 mm
- net GND: track 922.1 -> 920.6 mm
- net COL10: track 479.0 -> 480.1 mm
- net COL14: track 217.0 -> 217.8 mm
- net COL16: track 269.2 -> 269.9 mm
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Other:
- board text added: "DOMAIN-1"
- board text added: "DOMAIN-1 Mainboard PCB Rev 1.0 3/1/2022"
