File: DOMAIN-1_Upper-Board/DOMAIN-1_Upper-Board.sch (KiCad schematic (older format))
At the start: 53 parts

Commit message: Finished Upperboard
Parts:
- added C1, C2, C3, C4: 0.1uF, Capacitor_SMD:C_0603_1608Metric, symbol Device:C_Small
- D1, D10, D11, D12, D13, D14, D15, D16, D17, D18, D19, D2, D20, D21, D22, D23, D24, D3, D4, D5, D6, D7, D8, D9: renamed from D?; footprint (none) -> Diode_SMD:D_SOD-123
- J1: renamed from J?; footprint (none) -> Connector_IDC:IDC-Header_2x10_P2.54mm_Horizontal
- K_F13, K_F14, K_F15, K_F16, K_F17, K_F18, K_F19, K_F20, K_F21, K_F22, K_F23, K_F24, K_F25, K_F26, K_F27, K_F28, K_F29, K_F30, K_F31, K_F32, K_F33, K_F34, K_F35, K_F36: footprint (none) -> MX_Only:MXOnly-1.75U-Hotswap
- LED1, LED2, LED3, LED4: renamed from LED?; footprint (none) -> WS2812B:WS2812B
Connections:
- net +5V: now also J1.1 (Pin_1), C1.1, C2.1, C3.1, C4.1; no longer J1.17 (Pin_17)
- net COL10: now also J1.16 (Pin_16); no longer J1.3 (Pin_3)
- net COL11: now also J1.4 (Pin_4); no longer J1.2 (Pin_2)
- net COL12: now also J1.6 (Pin_6); no longer J1.4 (Pin_4)
- net COL13: now also J1.8 (Pin_8); no longer J1.6 (Pin_6)
- net COL14: now also J1.10 (Pin_10); no longer J1.8 (Pin_8)
- net COL15: now also J1.12 (Pin_12); no longer J1.10 (Pin_10)
- net COL16: now also J1.14 (Pin_14); no longer J1.12 (Pin_12)
- net COL17: now also J1.9 (Pin_9); no longer J1.14 (Pin_14)
- net COL18: now also J1.7 (Pin_7); no longer J1.16 (Pin_16)
- net COL19: now also J1.5 (Pin_5); no longer J1.18 (Pin_18)
- net COL20: now also J1.3 (Pin_3); no longer J1.20 (Pin_20)
- net COL9: now also J1.20 (Pin_20); no longer J1.5 (Pin_5)
- net GND: now also C1.2, C2.2, C3.2, C4.2
- net RGBLED_toUpperBoard: now also J1.2 (Pin_2); no longer J1.1 (Pin_1)
- net ROW6: now also J1.13 (Pin_13); no longer J1.7 (Pin_7)
- net ROW7: now also J1.15 (Pin_15); no longer J1.9 (Pin_9)
