File: DOMAIN-1_Upper-Board/DOMAIN-1_Upper-Board.kicad_pcb (KiCad board)
At the start: 2 copper layers, 441.5 x 51.9 mm, 57 parts, among them J1 Conn_02x10_Odd_Even

Commit message: Generated gerber files
Other:
- board text added: "DOMAIN-1"
- board text added: "DOMAIN-1 Upper Board PCB Rev 1.0 3/1/2022"
Changed lines of the file:
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@@
   (general
     (thickness 1.6)
-    (drawings 210)
+    (drawings 214)
     (tracks 460)
     (zones 0)
@@
     (solder_mask_min_width 0.25)
     (aux_axis_origin 0 0)
-    (visible_elements FFFFFF7F)
+    (visible_elements 7FFFFFFF)
     (pcbplotparams
-      (layerselection 0x010fc_ffffffff)
+      (layerselection 0x010f0_ffffffff)
       (usegerberextensions false)
       (usegerberattributes false)
@@
       (outputformat 1)
       (mirror false)
-      (drillshape 1)
+      (drillshape 0)
       (scaleselection 1)
-      (outputdirectory ""))
+      (outputdirectory "Gerbers/"))
   )
   (net 0 "")
@@
     )
   )
+  (gr_text "DOMAIN-1 Upper Board PCB Rev 1.0 3/1/2022" (at 409.702 169.672) (layer B.SilkS)
+    (effects (font (size 1 1) (thickness 0.15)) (justify mirror))
+  )
+  (gr_text DOMAIN-1 (at 130.302 166.751) (layer B.SilkS)
+    (effects (font (size 7 7) (thickness 0.7)) (justify mirror))
+  )
+  (gr_text "DOMAIN-1 Upper Board PCB Rev 1.0 3/1/2022" (at 409.702 169.672) (layer F.SilkS)
+    (effects (font (size 1 1) (thickness 0.15)))
+  )
+  (gr_text DOMAIN-1 (at 130.048 166.751) (layer F.SilkS)
+    (effects (font (size 7 7) (thickness 0.7)))
+  )
   (gr_line (start 59.055 164.338) (end 59.055 169.545) (layer Edge.Cuts) (width 0.05))
